File: kicad/and-gates-p1/and-gates-p1.kicad_sch (KiCad schematic)
At the start: 4 parts

Commit message: Update and export schematics
Other:
- note added: "The LED will light up when both inputs are pressed. This doesn't make this a "gate". In a gate inputs should be controlled with a signal, not requiring human intervention Also, the output here (if we consider the spot before D1 as the output) is floating when no buttons are pressed, usually you'd want a low value around 0V"
- company: (none) -> Silicon Chronicles
- title: Building AND gates the wrong way: Intro -> Intro
Changed lines of the file:
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@@
 	(paper "A5")
 	(title_block
-		(title "Building AND gates the wrong way: Intro")
+		(title "Intro")
+		(date "2024-04-28")
+		(company "Silicon Chronicles")
+		(comment 1 "Building AND gates the wrong way")
+		(comment 2 "Part I")
 	)
 	(wire
@@
 		)
 	)
+	(text "The LED will light up when both inputs are pressed.\n\nThis doesn't make this a \"gate\". In a gate inputs should\nbe controlled with a signal, not requiring human intervention\n\nAlso, the output here (if we consider the spot before D1 as the output)\nis floating when no buttons are pressed, usually you'd want a low\nvalue around 0V"
+		(exclude_from_sim no)
+		(at 97.536 34.036 0)
+		(effects
+			(font
+				(size 1.524 1.524)
+			)
+			(justify left)
+		)
+	)
