File: kicad/and-gates-p4/and-gates-p4.kicad_sch (KiCad schematic)
At the start: 42 parts, among them Q1 PN2222A, Q10 PN2222A, Q11 PN2222A, Q12 PN2222A, Q2 PN2222A, Q3 PN2222A, Q4 PN2222A, Q5 PN2222A, Q6 PN2222A, Q7 PN2222A, Q8 PN2222A, Q9 PN2222A

Commit message: Add extra schematics
Other:
- added sheet Additional diagrams (extras.kicad_sch)
Changed lines of the file:
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@@
+		)
+	)
+	(sheet
+		(at 25.4 172.72)
+		(size 12.7 3.81)
+		(fields_autoplaced yes)
+		(stroke
+			(width 0.1524)
+			(type solid)
+		)
+		(fill
+			(color 0 0 0 0.0000)
+		)
+		(property "Sheetname" "Additional diagrams"
+			(at 25.4 172.0084 0)
+			(effects
+				(font
+					(size 1.27 1.27)
+				)
+				(justify left bottom)
+			)
+		)
+		(property "Sheetfile" "extras.kicad_sch"
+			(at 25.4 177.1146 0)
+			(effects
+				(font
+					(size 1.27 1.27)
+				)
+				(justify left top)
+			)
+		)
+		(instances
+			(project "and-gates-p4"
+				(path "/66407854-f767-4de9-b271-5a41632efb59"
+					(page "2")
+				)
+			)
 		)
 	)
